Commit message: add mid360 urdf/xacro

File: urdf/go2_description.urdf.xacro (robot description, xacro)
@@ -15,5 +15,5 @@
       <origin xyz="0 0 0" rpy="0 0 0" />
       <geometry>
-         <mesh filename="file://$(find go2_description)/dae/base.dae" scale="1 1 1"/>
+         <mesh filename="package://go2_description/dae/base.dae" scale="1 1 1"/>
       </geometry>
       <material

File: urdf/leg.urdf.xacro (robot description, xacro)
@@ -29,5 +29,5 @@
         <origin xyz="0 0 0" rpy="0 0 0" />
         <geometry>
-          <mesh filename="file://$(find go2_description)/dae/hip.dae" scale="1 1 1"/>
+          <mesh filename="package://go2_description/dae/hip.dae" scale="1 1 1"/>
         </geometry>
         <material
@@ -63,8 +63,8 @@
         <geometry>
           <xacro:if value="${(name == LF) or (name == LR)}">
-            <mesh filename="file://$(find go2_description)/dae/thigh.dae" scale="1 1 1"/>
+            <mesh filename="package://go2_description/dae/thigh.dae" scale="1 1 1"/>
           </xacro:if>
            <xacro:if value="${(name == RF) or (name == RR)}">
-            <mesh filename="file://$(find go2_description)/dae/thigh_mirror.dae" scale="1 1 1"/>
+            <mesh filename="package://go2_description/dae/thigh_mirror.dae" scale="1 1 1"/>
           </xacro:if>
         </geometry>
@@ -101,8 +101,8 @@
         <geometry>
           <xacro:if value="${(name == LF) or (name == LR)}">
-            <mesh filename="file://$(find go2_description)/dae/calf.dae" scale="1 1 1"/>
+            <mesh filename="package://go2_description/dae/calf.dae" scale="1 1 1"/>
           </xacro:if>
            <xacro:if value="${(name == RF) or (name == RR)}">
-            <mesh filename="file://$(find go2_description)/dae/calf_mirror.dae" scale="1 1 1"/>
+            <mesh filename="package://go2_description/dae/calf_mirror.dae" scale="1 1 1"/>
           </xacro:if>
         </geometry>
@@ -137,5 +137,5 @@
         <origin xyz="0 0 0" rpy="0 0 0" />
         <geometry>
-          <mesh filename="file://$(find go2_description)/dae/foot.dae" scale="1 1 1"/>
+          <mesh filename="package://go2_description/dae/foot.dae" scale="1 1 1"/>
         </geometry>
         <material
