Commit message: Changed TF name

File: urdf/go2_description_airy1.urdf (robot description, URDF)
Before this commit: robot go2_description, 30 links, 29 joints
Links:
- removed link Go2_FL_calf
- removed link Go2_FL_calflower
- removed link Go2_FL_calflower1
- removed link Go2_FL_foot
- removed link Go2_FL_hip
- removed link Go2_FL_thigh
- removed link Go2_FR_calf
- removed link Go2_FR_calflower
- removed link Go2_FR_calflower1
- removed link Go2_FR_foot
- removed link Go2_FR_hip
- removed link Go2_FR_thigh
- removed link Go2_Head_lower
- removed link Go2_Head_upper
- removed link Go2_RL_calf
- removed link Go2_RL_calflower
- removed link Go2_RL_calflower1
- removed link Go2_RL_foot
- removed link Go2_RL_hip
- removed link Go2_RL_thigh
- removed link Go2_RR_calf
- removed link Go2_RR_calflower
- removed link Go2_RR_calflower1
- removed link Go2_RR_foot
- removed link Go2_RR_hip
- removed link Go2_RR_thigh
- removed link Go2_base_link
- removed link Go2_imu
- removed link Go2_rslidar_points
- removed link Go2_utlidar_lidar
- added link FL_calf, mass 0.154; collision cylinder length=0.12 radius=0.012; visual mesh filename=package://go2_description/dae/calf.dae
- added link FL_calflower; collision cylinder length=0.065 radius=0.011
- added link FL_calflower1; collision cylinder length=0.03 radius=0.0155
- added link FL_foot, mass 0.04; collision sphere radius=0.022; visual mesh filename=package://go2_description/dae/foot.dae
- added link FL_hip, mass 0.678; collision cylinder length=0.04 radius=0.046; visual mesh filename=package://go2_description/dae/hip.dae
- added link FL_thigh, mass 1.152; collision box size=0.213 0.0245 0.034; visual mesh filename=package://go2_description/dae/thigh.dae
- added link FR_calf, mass 0.154; collision cylinder length=0.12 radius=0.013; visual mesh filename=package://go2_description/dae/calf_mirror.dae
- added link FR_calflower; collision cylinder length=0.065 radius=0.011
- added link FR_calflower1; collision cylinder length=0.03 radius=0.0155
- added link FR_foot, mass 0.04; collision sphere radius=0.022; visual mesh filename=package://go2_description/dae/foot.dae
- added link FR_hip, mass 0.678; collision cylinder length=0.04 radius=0.046; visual mesh filename=package://go2_description/dae/hip.dae
- added link FR_thigh, mass 1.152; collision box size=0.213 0.0245 0.034; visual mesh filename=package://go2_description/dae/thigh_mirror.dae
- added link Head_lower, mass 0.001; collision sphere radius=0.047
- added link Head_upper, mass 0.001; collision cylinder length=0.09 radius=0.05
- added link RL_calf, mass 0.154; collision cylinder length=0.12 radius=0.013; visual mesh filename=package://go2_description/dae/calf.dae
- added link RL_calflower; collision cylinder length=0.065 radius=0.011
- added link RL_calflower1; collision cylinder length=0.03 radius=0.0155
- added link RL_foot, mass 0.04; collision sphere radius=0.022; visual mesh filename=package://go2_description/dae/foot.dae
- added link RL_hip, mass 0.678; collision cylinder length=0.04 radius=0.046; visual mesh filename=package://go2_description/dae/hip.dae
- added link RL_thigh, mass 1.152; collision box size=0.213 0.0245 0.034; visual mesh filename=package://go2_description/dae/thigh.dae
- added link RR_calf, mass 0.154; collision cylinder length=0.12 radius=0.013; visual mesh filename=package://go2_description/dae/calf_mirror.dae
- added link RR_calflower; collision cylinder length=0.065 radius=0.011
- added link RR_calflower1; collision cylinder length=0.03 radius=0.0155
- added link RR_foot, mass 0.04; collision sphere radius=0.022; visual mesh filename=package://go2_description/dae/foot.dae
- added link RR_hip, mass 0.678; collision cylinder length=0.04 radius=0.046; visual mesh filename=package://go2_description/dae/hip.dae
- added link RR_thigh, mass 1.152; collision box size=0.213 0.0245 0.034; visual mesh filename=package://go2_description/dae/thigh_mirror.dae
- added link base_link, mass 6.921; collision box size=0.3762 0.0935 0.114; visual mesh filename=package://go2_description/dae/base.dae
- added link imu, mass 0
- added link rslidar_points, mass 0.001; collision box size=0.0 0.0 0.0
- added link utlidar_lidar, mass 0
Joints:
- removed joint Go2_FL_calf_joint
- removed joint Go2_FL_calflower1_joint
- removed joint Go2_FL_calflower_joint
- removed joint Go2_FL_foot_joint
- removed joint Go2_FL_hip_joint
- removed joint Go2_FL_thigh_joint
- removed joint Go2_FR_calf_joint
- removed joint Go2_FR_calflower1_joint
- removed joint Go2_FR_calflower_joint
- removed joint Go2_FR_foot_joint
- removed joint Go2_FR_hip_joint
- removed joint Go2_FR_thigh_joint
- removed joint Go2_Head_lower_joint
- removed joint Go2_Head_upper_joint
- removed joint Go2_RL_calf_joint
- removed joint Go2_RL_calflower1_joint
- removed joint Go2_RL_calflower_joint
- removed joint Go2_RL_foot_joint
- removed joint Go2_RL_hip_joint
- removed joint Go2_RL_thigh_joint
- removed joint Go2_RR_calf_joint
- removed joint Go2_RR_calflower1_joint
- removed joint Go2_RR_calflower_joint
- removed joint Go2_RR_foot_joint
- removed joint Go2_RR_hip_joint
- removed joint Go2_RR_thigh_joint
- removed joint Go2_imu_joint
- removed joint Go2_rslidar_joint
- removed joint Go2_utlidar_lidar_joint
- added joint FL_calf_joint: type revolute, parent FL_thigh, child FL_calf, origin xyz=0 0 -0.213 rpy=0 0 0, axis 0 1 0, limit lower=-2.7227 upper=-0.83776 effort=45.43 velocity=15.70
- added joint FL_calflower1_joint: type fixed, parent FL_calflower, child FL_calflower1, origin xyz=-0.01 0 -0.04 rpy=0 0.48 0, axis 0 0 0
- added joint FL_calflower_joint: type fixed, parent FL_calf, child FL_calflower, origin xyz=0.020 0 -0.148 rpy=0 0.05 0, axis 0 0 0
- added joint FL_foot_joint: type fixed, parent FL_calf, child FL_foot, origin xyz=0 0 -0.213 rpy=0 0 0, axis 0 0 0
- added joint FL_hip_joint: type revolute, parent base_link, child FL_hip, origin xyz=0.1934 0.0465 0 rpy=0 0 0, axis 1 0 0, limit lower=-1.0472 upper=1.0472 effort=23.7 velocity=30.1
- added joint FL_thigh_joint: type revolute, parent FL_hip, child FL_thigh, origin xyz=0 0.0955 0 rpy=0 0 0, axis 0 1 0, limit lower=-1.5708 upper=3.4907 effort=23.7 velocity=30.1
- added joint FR_calf_joint: type revolute, parent FR_thigh, child FR_calf, origin xyz=0 0 -0.213 rpy=0 0 0, axis 0 1 0, limit lower=-2.7227 upper=-0.83776 effort=45.43 velocity=15.70
- added joint FR_calflower1_joint: type fixed, parent FR_calflower, child FR_calflower1, origin xyz=-0.01 0 -0.04 rpy=0 0.48 0, axis 0 0 0
- added joint FR_calflower_joint: type fixed, parent FR_calf, child FR_calflower, origin xyz=0.020 0 -0.148 rpy=0 0.05 0, axis 0 0 0
- added joint FR_foot_joint: type fixed, parent FR_calf, child FR_foot, origin xyz=0 0 -0.213 rpy=0 0 0, axis 0 0 0
- added joint FR_hip_joint: type revolute, parent base_link, child FR_hip, origin xyz=0.1934 -0.0465 0 rpy=0 0 0, axis 1 0 0, limit lower=-1.0472 upper=1.0472 effort=23.7 velocity=30.1
- added joint FR_thigh_joint: type revolute, parent FR_hip, child FR_thigh, origin xyz=0 -0.0955 0 rpy=0 0 0, axis 0 1 0, limit lower=-1.5708 upper=3.4907 effort=23.7 velocity=30.1
- added joint Head_lower_joint: type fixed, parent Head_upper, child Head_lower, origin xyz=0.008 0 -0.07 rpy=0 0 0, axis 0 0 0
- added joint Head_upper_joint: type fixed, parent base_link, child Head_upper, origin xyz=0.285 0 0.01 rpy=0 0 0, axis 0 0 0
- added joint RL_calf_joint: type revolute, parent RL_thigh, child RL_calf, origin xyz=0 0 -0.213 rpy=0 0 0, axis 0 1 0, limit lower=-2.7227 upper=-0.83776 effort=45.43 velocity=15.70
- added joint RL_calflower1_joint: type fixed, parent RL_calflower, child RL_calflower1, origin xyz=-0.01 0 -0.04 rpy=0 0.48 0, axis 0 0 0
- added joint RL_calflower_joint: type fixed, parent RL_calf, child RL_calflower, origin xyz=0.020 0 -0.148 rpy=0 0.05 0, axis 0 0 0
- added joint RL_foot_joint: type fixed, parent RL_calf, child RL_foot, origin xyz=0 0 -0.213 rpy=0 0 0, axis 0 0 0
- added joint RL_hip_joint: type revolute, parent base_link, child RL_hip, origin xyz=-0.1934 0.0465 0 rpy=0 0 0, axis 1 0 0, limit lower=-1.0472 upper=1.0472 effort=23.7 velocity=30.1
- added joint RL_thigh_joint: type revolute, parent RL_hip, child RL_thigh, origin xyz=0 0.0955 0 rpy=0 0 0, axis 0 1 0, limit lower=-0.5236 upper=4.5379 effort=23.7 velocity=30.1
- added joint RR_calf_joint: type revolute, parent RR_thigh, child RR_calf, origin xyz=0 0 -0.213 rpy=0 0 0, axis 0 1 0, limit lower=-2.7227 upper=-0.83776 effort=45.43 velocity=15.70
- added joint RR_calflower1_joint: type fixed, parent RR_calflower, child RR_calflower1, origin xyz=-0.01 0 -0.04 rpy=0 0.48 0, axis 0 0 0
- added joint RR_calflower_joint: type fixed, parent RR_calf, child RR_calflower, origin xyz=0.020 0 -0.148 rpy=0 0.05 0, axis 0 0 0
- added joint RR_foot_joint: type fixed, parent RR_calf, child RR_foot, origin xyz=0 0 -0.213 rpy=0 0 0, axis 0 0 0
- added joint RR_hip_joint: type revolute, parent base_link, child RR_hip, origin xyz=-0.1934 -0.0465 0 rpy=0 0 0, axis 1 0 0, limit lower=-1.0472 upper=1.0472 effort=23.7 velocity=30.1
- added joint RR_thigh_joint: type revolute, parent RR_hip, child RR_thigh, origin xyz=0 -0.0955 0 rpy=0 0 0, axis 0 1 0, limit lower=-0.5236 upper=4.5379 effort=23.7 velocity=30.1
- added joint imu_joint: type fixed, parent base_link, child imu, origin xyz=-0.02557 0 0.04232 rpy=0 0 0, axis 0 0 0
- added joint rslidar_joint: type fixed, parent rslidar_points, child base_link, origin xyz=-0.15 0.0 -0.3 rpy=0.0 -0.6681 0.0
- added joint utlidar_lidar_joint: type fixed, parent base_link, child utlidar_lidar, origin xyz=0.28945 0 -0.046825 rpy=0 2.8782 0, axis 0 0 0
